File: esp32c3-iot-client-board.kicad_pcb (KiCad board)
At the start: 2 copper layers, 38.1 x 49.5 mm, 32 parts, among them J1 Prog, J2 USB2.0_C_v3, M1 M2-Hole, M2 M2-Hole, M3 M2-Hole, M4 M2-Hole, SW1 G3, SW2 BOOT, SW3 RST, U1 ESP32-C3-WROOM-02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

Commit message: up
Parts:
- removed U3: CH213K, Package_TO_SOT_SMD:SOT-23
- added R5: 10k, $74th:Capacitor_0805_2012, B.Cu at (136.4, 81.9)
- added R6: 10k, $74th:Capacitor_0805_2012, B.Cu at (136.4, 83.9)
- added R7: 10k, $74th:Capacitor_0805_2012, B.Cu at (143.8, 115.6)
- added R8: 42k, $74th:Capacitor_0805_2012, B.Cu at (143.7, 113.5)
- added U4: CH217K, Package_TO_SOT_SMD:SOT-23-6, B.Cu at (152.7, 105.7)
- D1: value WS2812B -> SK6812MINI; footprint LED_SMD:LED_WS2812B_PLCC4_5.0x5.0mm_P3.2mm -> $74th:YS-SK6812MINI-E-BACK-RIGHT; moved to B.Cu
- JP1, JP2, JP3: footprint Jumper:SolderJumper-3_P1.3mm_Open_RoundedPad1.0x1.5mm -> $74th:VCC_Selector_Jumper
- moved U2 5.21 mm to (156.3, 96.4)
- moved G*** 3.97 mm to (143.8, 79.9)
- moved C1 3.11 mm to (152.2, 79.3)
- moved C3 2.55 mm to (152.1, 83.8)
- moved C2 2.55 mm to (152.2, 81.3)
- moved D1 2.41 mm to (148.8, 96.0), turned to -90 degrees
- moved R1 2.05 mm to (152.1, 85.9)
- moved R2 1.55 mm to (152.1, 87.9)
- moved U1 0.81 mm to (155.3, 82.9)
Routing:
- net GND: track 48.9 -> 31.9 mm, vias 51 -> 61
- net Net-(U4-EN#): track 0.00 -> 15.8 mm
- net Net-(U4-ISET): track 0.00 -> 14.0 mm
- net Net-(CH1-VCC): track 8.37 -> 18.8 mm, vias 0 -> 1
- net +5V: track 76.3 -> 85.5 mm, vias 5 -> 6
- net /RX: track 77.5 -> 72.2 mm
- net /LED: track 23.4 -> 27.8 mm, vias 2 -> 3
- net /TX: track 75.0 -> 71.2 mm
- net /G0: track 38.7 -> 36.5 mm, vias 0 -> 3
- net /EN: track 63.8 -> 65.7 mm
- net /USBD-: track 44.9 -> 46.6 mm
- net /G5: track 36.9 -> 35.5 mm
- net Net-(J2-VBUS): track 18.8 -> 20.0 mm
- net /G1: track 35.9 -> 34.7 mm, vias 0 -> 1
- net /G4: track 41.5 -> 40.4 mm
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Other:
- board text added: "G2"
- board text added: "G4"
- board text added: "I2C PullUp"
- board text added: "v1.1.0"
- board text removed: "C4"
- board text removed: "v1.0.0"
