File: esp32c3-iot-client-board.kicad_sch (KiCad schematic)
At the start: 25 parts, among them J1 Prog, J2 USB2.0_C_v3, SW1 G3, SW2 BOOT, SW3 RST, U1 ESP32-C3-WROOM-02, U2 AMS1117-3.3, U3 CH213K

Commit message: up
Parts:
- removed D1: WS2812B, LED_SMD:LED_WS2812B_PLCC4_5.0x5.0mm_P3.2mm, symbol LED:WS2812B
- removed U3: CH213K, Package_TO_SOT_SMD:SOT-23, symbol $74th:CH213K-Ideal_Diode_for_USB_Power
- added D1: SK6812MINI, $74th:YS-SK6812MINI-E-BACK-RIGHT, symbol $74th:SK6812MINI
- added R5, R6, R7: 10k, $74th:Capacitor_0805_2012, symbol Device:R
- added R8: 42k, $74th:Capacitor_0805_2012, symbol Device:R
- added U4: CH217K, Package_TO_SOT_SMD:SOT-23-6, symbol $74th:CH217K-USB_Power_Limit_Switch
- JP1, JP2, JP3: footprint Jumper:SolderJumper-3_P1.3mm_Open_RoundedPad1.0x1.5mm -> $74th:VCC_Selector_Jumper
Connections:
- net +5V: now also D1.1 (VDD), U4.1 (VOUT)
- net G0: now also R6.2
- net G1: now also R5.2
- net GND: now also D1.3 (GND), R7.2, R8.2, U4.2 (GND)
- net LED: now also D1.4 (DIN)
- net at CH1.3 (VCC), JP1.2 (C): now also R5.1, R6.1
- net at F1.2, J2.1 (VBUS): now also U4.6 (VIN)
- new net: R7.1, U4.4 (EN#)
- new net: R8.1, U4.5 (ISET)
- no-connect marks 4 -> 5
Other:
- moved on the sheet: C4, C5, CH1, CH2, CH3, F1, JP1, JP2, JP3, R3, R4, U2
