File: pcb-kicad/esp32c3-iot-client-board.kicad_pcb (KiCad board)
At the start: 2 copper layers, 38.1 x 49.5 mm, 36 parts, among them J1 Prog, J2 USB2.0_C_v3, M1 M2-Hole, M2 M2-Hole, M3 M2-Hole, M4 M2-Hole, SW1 G3, SW2 BOOT, SW3 RST, U1 ESP32-C3-WROOM-02, U2 AMS1117-3.3, U4 CH217K

Commit message: v1.1.1
Parts:
- F1: value Polyfuse -> KT6-1100SMDI(NC)
- R5, R6: value 10k -> 1k(NC)
Connections:
- D1 pad 1: +5V -> +3V3
Routing:
- net +5V: track 85.5 -> 76.0 mm, vias 6 -> 4
- net +3V3: track 82.7 -> 85.6 mm
Other:
- board text added: "v1.1.1"
- board text removed: "v1.1.0"

Commit message: v1.2.0
Parts:
- removed F1: KT6-1100SMDI(NC), $74th:Fuse_1812_4532Metric_Pad1.30x3.40mm_HandSolder
- added C3: 10u, $74th:Capacitor_0805_2012, B.Cu at (142.6, 82.4)
- added C6: 10u, $74th:Capacitor_0805_2012, B.Cu at (142.3, 96.5)
- added C8: 10u, $74th:Capacitor_0805_2012, B.Cu at (142.3, 110.0)
- added R6: 27.4, $74th:Capacitor_0805_2012, B.Cu at (163.2, 109.0)
- added R7: 27.4, $74th:Capacitor_0805_2012, B.Cu at (163.2, 111.0)
- R8: value 42k -> 56k
- moved G*** 21.3 mm to (136.4, 99.9)
- moved R9 2.18 mm to (162.4, 114.8)
- moved SW3 1.00 mm to (162.9, 114.0)
- moved JP2 0.87 mm to (141.7, 101.2)
- moved SW2 0.82 mm to (162.8, 105.9)
- moved JP1 0.79 mm to (142.0, 86.9)
- moved JP3 0.63 mm to (142.0, 114.8)
- moved CH1 0.12 mm to (140.8, 81.0)
- renumbered C3 to C4, C4 to C5, C5 to C7, R5 to R1, R7 to R10, R6 to R2, R1 to R3, R2 to R4, R3 to R5, R4 to R9, U4 to U3
Connections:
- CH2 pad 1: /RX -> /G6
- CH2 pad 2: /TX -> /G7
- U1 pad 13: /USBD- -> Net-(U1-GPIO18/USB_D-)
- U1 pad 14: /USBD+ -> Net-(U1-GPIO19/USB_D+)
- U1 pad 5: unconnected-(U1-GPIO6-Pad5) -> /G6
- U1 pad 6: unconnected-(U1-GPIO7-Pad6) -> /G7
Routing:
- net /RX: track 72.2 -> 11.4 mm, vias 2 -> 1
- net /TX: track 71.2 -> 13.3 mm, vias 2 -> 1
- net /G7: track 0.00 -> 40.2 mm, vias 0 -> 2
- net /G6: track 0.00 -> 37.4 mm, vias 0 -> 2
- net /USBD+: track 46.3 -> 12.7 mm, vias 3 -> 2
- net Net-(U1-GPIO19/USB_D+): track 0.00 -> 32.1 mm, vias 0 -> 1
- net /USBD-: track 46.6 -> 14.6 mm, vias 2 -> 1
- net Net-(U1-GPIO18/USB_D-): track 0.00 -> 30.2 mm, vias 0 -> 1
- net GND: track 31.9 -> 44.7 mm, vias 61 -> 109
- net +3V3: track 85.6 -> 93.5 mm, vias 3 -> 4
- net Net-(J2-CC2): track 11.5 -> 15.1 mm, vias 1 -> 3
- net +5V: track 76.0 -> 77.7 mm
- net Net-(CH3-VCC): track 8.88 -> 10.5 mm, vias 0 -> 2
- net /BOOT: track 37.9 -> 39.4 mm
- net /EN: track 65.7 -> 67.2 mm
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Other:
- board text added: "R/8"
- board text added: "T/7"
- board text added: "v1.2.0"
- board text removed: "R/20"
- board text removed: "T/21"
- board text removed: "v1.1.1"
