File: pcb-kicad/esp32c3-iot-client-board.kicad_sch (KiCad schematic)
At the start: 29 parts, among them J1 Prog, J2 USB2.0_C_v3, SW1 G3, SW2 BOOT, SW3 RST, U1 ESP32-C3-WROOM-02, U2 AMS1117-3.3, U4 CH217K

Commit message: update document
Parts:
- F1: value Polyfuse -> KT6-1100SMDI(NC)
- R5, R6: value 10k -> 1k(NC)
Other:
- title: (none) -> ESP32C3 IoT Server
- moved on the sheet: CH1, JP1, R5, R6

Commit message: v1.1.1
Connections:
- net +3V3: now also D1.1 (VDD)
- net +5V: no longer D1.1 (VDD)
Changed lines of the file:
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@@
   (title_block
     (title "ESP32C3 IoT Server")
+    (rev "1.1.1")
   )
   (junction (at 20.32 55.88) (diameter 0) (color 0 0 0 0)
@@
     )
   )
-  (symbol (lib_id "power:+5V") (at 256.54 127 0) (unit 1)
-    (in_bom yes) (on_board yes) (dnp no) (fields_autoplaced)
-    (property "Reference" "#PWR029" (at 256.54 130.81 0)
-      (effects (font (size 1.27 1.27)) hide)
-    )
-    (property "Value" "+5V" (at 256.54 121.92 0)
-      (effects (font (size 1.27 1.27)))
-    )
-    (property "Footprint" "" (at 256.54 127 0)
-      (effects (font (size 1.27 1.27)) hide)
-    )
-    (property "Datasheet" "" (at 256.54 127 0)
-      (effects (font (size 1.27 1.27)) hide)
-    )
-    (pin "1")
-    (instances
-      (project "esp32c3-iot-client-board"
-        (path "/2360abc4-b955-42fd-b995-e0b25dda0008"
-          (reference "#PWR029") (unit 1)
-        )
-      )
-    )
-  )
   (symbol (lib_id "Device:R") (at 191.77 72.39 0) (unit 1)
     (in_bom yes) (on_board yes) (dnp no) (fields_autoplaced)
@@
         )
       )
+    )
+  )
+  (symbol (lib_id "power:+3V3") (at 256.54 127 0) (unit 1)
+    (in_bom yes) (on_board yes) (dnp no) (fields_autoplaced)
+    (property "Reference" "#PWR029" (at 256.54 130.81 0)
+      (effects (font (size 1.27 1.27)) hide)
+    )
+    (property "Value" "+3V3" (at 256.54 121.92 0)
+      (effects (font (size 1.27 1.27)))
+    )
+    (property "Footprint" "" (at 256.54 127 0)
+      (effects (font (size 1.27 1.27)) hide)
+    )
+    (property "Datasheet" "" (at 256.54 127 0)
+      (effects (font (size 1.27 1.27)) hide)
+    )
+    (pin "1")
+    (instances
+      (project "esp32c3-iot-client-board"
+        (path "/2360abc4-b955-42fd-b995-e0b25dda0008"
+          (reference "#PWR029") (unit 1)
+        )
+      )

Commit message: v1.2.0
Parts:
- removed F1: KT6-1100SMDI(NC), $74th:Fuse_1812_4532Metric_Pad1.30x3.40mm_HandSolder, symbol Device:Polyfuse
- added C3, C6, C8: 10u, $74th:Capacitor_0805_2012, symbol Device:C
- added R6, R7: 27.4, $74th:Capacitor_0805_2012, symbol Device:R
- R8: value 42k -> 56k
- renumbered C3 to C4, C4 to C5, C5 to C7, R5 to R1, R7 to R10, R6 to R2, R1 to R3, R2 to R4, R3 to R5, R4 to R9, U4 to U3
Connections:
- net GND: now also C3.2, C6.2, C8.2
- net RX: no longer CH2.1 (RX)
- net TX: no longer CH2.2 (TX)
- net USBD+: now also R7.1; no longer U1.14 (GPIO19/USB_D+)
- net USBD-: now also R6.1; no longer U1.13 (GPIO18/USB_D-)
- net at CH1.3 (VCC), JP1.2 (C), R1.1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: now also C3.1
- net at CH3.3 (VCC), JP3.2 (C): now also C8.1
- net at CH2.3 (VCC), JP2.2 (C): now also C6.1
- net G6: now reaches U1.5 (GPIO6)
- net G6: now also CH2.1 (RX)
- net G7: now reaches U1.6 (GPIO7)
- net G7: now also CH2.2 (TX)
- new net: R7.2, U1.14 (GPIO19/USB_D+)
- new net: R6.2, U1.13 (GPIO18/USB_D-)
- no-connect marks 5 -> 3
Other:
- moved on the sheet: C1, C2, CH1, CH2, CH3, JP1, JP2, JP3, R1, R2

Commit message: dumping register
Parts:
- R6, R7: value 27.4 -> 10
