File: modules-pcb/ir_send/ir_send.kicad_pcb (KiCad board)
At the start: 2 copper layers, 14 x 16.5 mm, 10 parts, among them M2 Hole_M2_2.0, Q1 2N7002

Commit message: esp32-s3
Parts:
- D1, D2: footprint LED_THT:LED_D3.0mm_Horizontal_O1.27mm_Z2.0mm -> 74th:PinOut_Pin_2_1GND
Other:
- board text added: "v1.0.1"
- board text removed: "v1.0.0"
