File: modules-pcb/ir_send/ir_send.kicad_sch (KiCad schematic)
At the start: 7 parts, among them Q1 2N7002

Commit message: esp32-s3
Parts:
- D1, D2: footprint LED_THT:LED_D3.0mm_Horizontal_O1.27mm_Z2.0mm -> 74th:PinOut_Pin_2_1GND
Changed lines of the file:
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@@
 	(title_block
 		(title "IR Grove")
-		(rev "1.0.0")
+		(rev "1.0.1")
 		(company "Atsushi Morimoto (@74th)")
 	)
@@
 			)
 		)
-		(property "Footprint" "LED_THT:LED_D3.0mm_Horizontal_O1.27mm_Z2.0mm"
+		(property "Footprint" "74th:PinOut_Pin_2_1GND"
 			(at 167.64 59.69 0)
 			(effects
@@
 			)
 		)
-		(property "Footprint" "LED_THT:LED_D3.0mm_Horizontal_O1.27mm_Z2.0mm"
+		(property "Footprint" "74th:PinOut_Pin_2_1GND"
 			(at 151.13 59.69 0)
 			(effects
